File: PCB/Keyboard-PCB.kicad_pcb (KiCad board)
At the start: 2 copper layers, 133.1 x 105.7 mm, 48 parts, among them J1 USB_C_Receptacle_USB2.0_16P, J2 USB_C_Receptacle_USB2.0_16P, SW1 SW_Push, SW10 SW_Push, SW11 SW_Push, SW12 SW_Push, SW13 SW_Push, SW14 SW_Push, SW15 SW_Push, SW16 SW_Push, SW17 SW_Push, SW18 SW_Push, SW19 SW_Push, SW2 SW_Push, SW20 SW_Push, SW21 SW_Push, SW3 SW_Push, SW4 SW_Push, SW5 SW_Push, SW6 SW_Push, SW7 SW_Push, SW8 SW_Push, SW9 SW_Push, U2 STM32WB55CCUx

Commit message: new hotswap footprints and adjustments
Parts:
- removed PS1: TAR5SB33_TE85L,F_, MyLibrary:SOT95P275X140-5N
- added D22: D, Diode_SMD:D_0805_2012Metric, B.Cu at (181.8, 63.9)
- added D23: D, Diode_SMD:D_0805_2012Metric, B.Cu at (181.8, 82.9)
- added D24: D, Diode_SMD:D_0805_2012Metric, B.Cu at (181.8, 101.9)
- added D25: D, Diode_SMD:D_0805_2012Metric, B.Cu at (200.8, 59.4)
- added D26: D, Diode_SMD:D_0805_2012Metric, B.Cu at (200.8, 78.4)
- added D27: D, Diode_SMD:D_0805_2012Metric, B.Cu at (200.8, 97.4)
- added D28: D, Diode_SMD:D_0805_2012Metric, B.Cu at (219.8, 50.9)
- added D29: D, Diode_SMD:D_0805_2012Metric, B.Cu at (219.8, 69.9)
- added D30: D, Diode_SMD:D_0805_2012Metric, B.Cu at (219.8, 88.9)
- added D31: D, Diode_SMD:D_0805_2012Metric, B.Cu at (238.8, 57.2)
- added D32: D, Diode_SMD:D_0805_2012Metric, B.Cu at (238.8, 76.2)
- added D33: D, Diode_SMD:D_0805_2012Metric, B.Cu at (238.8, 94.9)
- added D34: D, Diode_SMD:D_0805_2012Metric, B.Cu at (258.0, 62.9)
- added D35: D, Diode_SMD:D_0805_2012Metric, B.Cu at (257.8, 81.9)
- added D36: D, Diode_SMD:D_0805_2012Metric, B.Cu at (257.8, 100.9)
- added D37: D, Diode_SMD:D_0805_2012Metric, B.Cu at (276.8, 69.4)
- added D38: D, Diode_SMD:D_0805_2012Metric, B.Cu at (276.8, 88.4)
- added D39: D, Diode_SMD:D_0805_2012Metric, B.Cu at (276.8, 107.4)
- added D40: D, Diode_SMD:D_0805_2012Metric, B.Cu at (167.4, 125.7)
- added D41: D, Diode_SMD:D_0805_2012Metric, B.Cu at (190.2, 120.2)
- added D42: D, Diode_SMD:D_0805_2012Metric, B.Cu at (210.8, 120.0)
- added SW22: SW_Push, MyLibrary:MX100H, B.Cu at (173.5, 64.0)
- added SW23: SW_Push, MyLibrary:MX100H, B.Cu at (173.5, 83.0)
- added SW24: SW_Push, MyLibrary:MX100H, B.Cu at (173.5, 102.0)
- added SW25: SW_Push, MyLibrary:MX100H, B.Cu at (192.5, 59.5)
- added SW26: SW_Push, MyLibrary:MX100H, B.Cu at (192.5, 78.5)
- added SW27: SW_Push, MyLibrary:MX100H, B.Cu at (192.5, 97.5)
- added SW28: SW_Push, MyLibrary:MX100H, B.Cu at (211.5, 51.0)
- added SW29: SW_Push, MyLibrary:MX100H, B.Cu at (211.5, 70.0)
- added SW30: SW_Push, MyLibrary:MX100H, B.Cu at (211.5, 89.0)
- added SW31: SW_Push, MyLibrary:MX100H, B.Cu at (230.5, 57.0)
- added SW32: SW_Push, MyLibrary:MX100H, B.Cu at (230.5, 76.0)
- added SW33: SW_Push, MyLibrary:MX100H, B.Cu at (230.5, 95.0)
- added SW34: SW_Push, MyLibrary:MX100H, B.Cu at (249.5, 63.0)
- added SW35: SW_Push, MyLibrary:MX100H, B.Cu at (249.5, 82.0)
- added SW36: SW_Push, MyLibrary:MX100H, B.Cu at (249.5, 101.0)
- added SW37: SW_Push, MyLibrary:MX100H, B.Cu at (268.5, 69.5)
- added SW38: SW_Push, MyLibrary:MX100H, B.Cu at (268.5, 88.5)
- added SW39: SW_Push, MyLibrary:MX100H, B.Cu at (268.5, 107.5)
- added SW40: SW_Push, MyLibrary:MX100H, B.Cu at (161.1, 131.0)
- added SW41: SW_Push, MyLibrary:MX100H, B.Cu at (182.1, 121.7)
- added SW42: SW_Push, MyLibrary:MX100H, B.Cu at (202.5, 120.0)
- added U1: STM32WB55CCUx, Package_DFN_QFN:QFN-48-1EP_7x7mm_P0.5mm_EP5.6x5.6mm, F.Cu at (239.8, 135.5)
- D1, D10, D11, D12, D13, D14, D15, D16, D17, D18, D19, D2, D20, D21, D3, D4, D5, D6, D7, D8, D9: footprint Diode_SMD:Nexperia_CFP3_SOD-123W -> Diode_SMD:D_0805_2012Metric
- J1: moved to F.Cu
- SW1, SW10, SW11, SW12, SW13, SW14, SW15, SW16, SW17, SW18, SW19, SW2, SW20, SW21, SW3, SW4, SW5, SW6, SW7, SW8, SW9: footprint Button_Switch_Keyboard:SW_Cherry_MX_1.00u_PCB -> MyLibrary:MX100H; moved to B.Cu
- U2: value STM32WB55CCUx -> AMS1117-3.3; footprint Package_DFN_QFN:QFN-48-1EP_7x7mm_P0.5mm_EP5.6x5.6mm -> Package_TO_SOT_SMD:SOT-223-3_TabPin2; moved to F.Cu
- moved SW21 181.5 mm to (92.5, 120.0), turned to 180 degrees
- moved D21 168.6 mm to (100.8, 119.9)
- moved SW20 139.2 mm to (112.9, 121.7), turned to 170 degrees
- moved SW1 138.4 mm to (121.5, 64.0), turned to 180 degrees
- moved SW10 138.4 mm to (64.5, 57.0), turned to 180 degrees
- moved SW11 138.4 mm to (64.5, 76.0), turned to 180 degrees
- moved SW12 138.4 mm to (64.5, 95.0), turned to 180 degrees
- moved SW13 138.4 mm to (45.5, 63.0), turned to 180 degrees
- moved SW14 138.4 mm to (45.5, 82.0), turned to 180 degrees
- moved SW15 138.4 mm to (45.5, 101.0), turned to 180 degrees
- moved SW16 138.4 mm to (26.5, 69.5), turned to 180 degrees
- moved SW17 138.4 mm to (26.5, 88.5), turned to 180 degrees
- moved SW18 138.4 mm to (26.5, 107.5), turned to 180 degrees
- moved SW2 138.4 mm to (121.5, 83.0), turned to 180 degrees
- moved SW4 138.4 mm to (102.5, 59.5), turned to 180 degrees
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Connections:
- net column1 renamed /SwitchClusterLeft/Column1
- net column2 renamed /SwitchClusterLeft/Column2
- net column3 renamed /SwitchClusterLeft/Column3
- net column4 renamed /SwitchClusterLeft/Column4
- net column5 renamed /SwitchClusterLeft/Column5
- net column6 renamed /SwitchClusterLeft/Column6
- net column7 renamed /SwitchClusterLeft/Column7
- net row1 renamed /SwitchClusterLeft/Row1
- net row2 renamed /SwitchClusterLeft/Row2
- net row3 renamed /SwitchClusterLeft/Row3
- J1 pad A4: +5V -> VBUS
- J1 pad A9: +5V -> VBUS
- J1 pad B4: +5V -> VBUS
- J1 pad B9: +5V -> VBUS
- J2 pad A1: GND -> Net-(J2-GND-PadA1)
- J2 pad A12: GND -> Net-(J2-GND-PadA1)
- J2 pad A4: +5V -> Net-(J2-VBUS-PadA4)
- J2 pad A6: Net-(J2-D+-PadA6) -> unconnected-(J2-D+-PadA6)
- J2 pad A7: Net-(J2-D--PadA7) -> unconnected-(J2-D--PadA7)
- J2 pad A9: +5V -> Net-(J2-VBUS-PadA4)
- J2 pad B1: GND -> Net-(J2-GND-PadA1)
- J2 pad B12: GND -> Net-(J2-GND-PadA1)
- J2 pad B4: +5V -> Net-(J2-VBUS-PadA4)
- J2 pad B6: Net-(J2-D+-PadA6) -> unconnected-(J2-D+-PadB6)
- J2 pad B7: Net-(J2-D--PadA7) -> unconnected-(J2-D--PadB7)
- J2 pad B9: +5V -> Net-(J2-VBUS-PadA4)
- J2 pad SH: GND -> unconnected-(J2-SHIELD-PadSH)
Other:
- board outline removed

Commit message: Board Outline
Parts:
- moved J1 9.55 mm to (231.9, 131.6), turned to 180 degrees
Other:
- board outline added: 260 x 100.9 mm

Commit message: Basic Component Placement
Parts:
- added C1: 10uF, Capacitor_SMD:C_0402_1005Metric, B.Cu at (88.0, 108.0)
- added C10: 100nF, Capacitor_SMD:C_0402_1005Metric, B.Cu at (203.5, 99.1)
- added C11: 100nF, Capacitor_SMD:C_0402_1005Metric, B.Cu at (89.0, 104.5)
- added C12: 100nF, Capacitor_SMD:C_0402_1005Metric, B.Cu at (88.0, 104.5)
- added C13: 1uF, Capacitor_SMD:C_0402_1005Metric, B.Cu at (86.8, 104.5)
- added C14: 100n, Capacitor_SMD:C_0402_1005Metric, B.Cu at (88.5, 106.0)
- added C15: 100nF, Capacitor_SMD:C_0402_1005Metric, B.Cu at (206.8, 106.1)
- added C16: 100nF, Capacitor_SMD:C_0402_1005Metric, B.Cu at (207.8, 106.1)
- added C17: 1uF, Capacitor_SMD:C_0402_1005Metric, B.Cu at (209.0, 106.1)
- added C18: 100n, Capacitor_SMD:C_0402_1005Metric, B.Cu at (207.2, 104.5)
- added C19: 0.1uF, Capacitor_SMD:C_0402_1005Metric, B.Cu at (113.2, 112.0)
- added C2: 100nF, Capacitor_SMD:C_0402_1005Metric, B.Cu at (89.2, 108.0)
- added C20: 0.1uF, Capacitor_SMD:C_0402_1005Metric, B.Cu at (113.2, 109.5)
- added C21: 0.1uF, Capacitor_SMD:C_0402_1005Metric, B.Cu at (113.2, 108.2)
- added C22: 0.1uF, Capacitor_SMD:C_0402_1005Metric, B.Cu at (113.2, 110.8)
- added C3: 100nF, Capacitor_SMD:C_0402_1005Metric, B.Cu at (97.5, 99.8)
- added C4: 100nF, Capacitor_SMD:C_0402_1005Metric, B.Cu at (100.8, 108.0)
- added C5: 100nF, Capacitor_SMD:C_0402_1005Metric, B.Cu at (92.5, 111.5)
- added C6: 4.7uF, Capacitor_SMD:C_0402_1005Metric, B.Cu at (208.0, 102.6)
- added C7: 100nF, Capacitor_SMD:C_0402_1005Metric, B.Cu at (206.8, 102.6)
- added C8: 100nF, Capacitor_SMD:C_0402_1005Metric, B.Cu at (198.5, 110.8)
- added C9: 100nF, Capacitor_SMD:C_0402_1005Metric, B.Cu at (195.0, 102.6)
- added D43: SP0503BAHT, Package_TO_SOT_SMD:SOT-143, B.Cu at (126.5, 92.0)
- added J3: BOOT0, Connector_PinHeader_2.54mm:PinHeader_1x03_P2.54mm_Vertical, B.Cu at (137.5, 103.5)
- added J4: BOOT1, Connector_PinHeader_2.54mm:PinHeader_1x03_P2.54mm_Vertical, B.Cu at (133.8, 104.2)
- added J5: BOOT0, Connector_PinHeader_2.54mm:PinHeader_1x03_P2.54mm_Vertical, B.Cu at (161.5, 104.0)
- added J6: BOOT1, Connector_PinHeader_2.54mm:PinHeader_1x03_P2.54mm_Vertical, B.Cu at (157.8, 103.3)
- added J7: AudioJack4, MyLibrary:Jack_3.5mm_CUI_SJ1-3524N_Horizontal, B.Cu at (157.5, 113.5)
- added R5: 10k, Resistor_SMD:R_0805_2012Metric, B.Cu at (95.1, 111.8)
- added R6: 10k, Resistor_SMD:R_0805_2012Metric, B.Cu at (94.6, 99.2)
- added R7: 10k, Resistor_SMD:R_0805_2012Metric, B.Cu at (200.8, 98.8)
- added R8: 10k, Resistor_SMD:R_0805_2012Metric, B.Cu at (201.3, 111.2)
- added SW43: SW_Push, Button_Switch_SMD:SW_Push_1P1T_NO_CK_KMR2, B.Cu at (212.0, 103.0)
- added SW45: SW_Push, Button_Switch_SMD:SW_Push_1P1T_NO_CK_KMR2, B.Cu at (82.5, 104.0)
- added U3: STM32F103C6Tx, Package_QFP:LQFP-48_7x7mm_P0.5mm, B.Cu at (201.0, 105.0)
- J1, R1, R2, U2: moved to B.Cu
- J2: value USB_C_Receptacle_USB2.0_16P -> AudioJack4; footprint Connector_USB:USB_C_Receptacle_GCT_USB4085 -> MyLibrary:Jack_3.5mm_CUI_SJ1-3524N_Horizontal; moved to B.Cu
- U1: value STM32WB55CCUx -> STM32F103C6Tx; footprint Package_DFN_QFN:QFN-48-1EP_7x7mm_P0.5mm_EP5.6x5.6mm -> Package_QFP:LQFP-48_7x7mm_P0.5mm; moved to B.Cu
- moved U1 147.8 mm to (95.0, 105.5)
- moved U2 133.1 mm to (107.7, 109.0), turned to 180 degrees
- moved R2 124.7 mm to (126.1, 87.5)
- moved R1 124.3 mm to (126.1, 85.5), turned to 180 degrees
- moved J1 113.2 mm to (129.8, 82.8), turned to -80 degrees
- moved J2 90.8 mm to (137.8, 113.6), turned to -78 degrees
- moved D34 9.95 mm to (249.4, 68.0), turned to 0 degrees
- moved D33 9.87 mm to (230.4, 100.2), turned to 0 degrees
- moved D21 9.84 mm to (92.3, 125.0), turned to 0 degrees
- moved D17 9.76 mm to (26.6, 93.8), turned to 0 degrees
- moved D19 9.74 mm to (130.5, 134.9), turned to -40 degrees
- moved D25 9.73 mm to (192.4, 64.5), turned to 0 degrees
- moved D26 9.73 mm to (192.4, 83.5), turned to 0 degrees
- moved D27 9.73 mm to (192.4, 102.5), turned to 0 degrees
- moved D28 9.73 mm to (211.4, 56.0), turned to 0 degrees
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Connections:
- U1 pad 20: +3.3V -> /BOOT1
- U1 pad 23: unconnected-(U1-VDDRF-Pad23) -> GND
- U1 pad 24: unconnected-(U1-OSC_OUT-Pad24) -> +3.3V
- U1 pad 35: +3.3V -> GND
- U1 pad 36: unconnected-(U1-PA10-Pad36) -> +3.3V
- U1 pad 44: unconnected-(U1-PB4-Pad44) -> /BOOT0
- U1 pad 47: unconnected-(U1-PB7-Pad47) -> GND
- U1 pad 7: unconnected-(U1-NRST-Pad7) -> /NRST
- U1 pad 8: unconnected-(U1-VDDA-Pad8) -> GND
- U1 pad 9: unconnected-(U1-PA0-Pad9) -> +3.3V
- U2 pad 1: unconnected-(U2-GND-Pad1) -> GND
- U2 pad 2: unconnected-(U2-VO-Pad2) -> +3.3V
- U2 pad 3: unconnected-(U2-VI-Pad3) -> VBUS
Other:
- board text added: "0"
- board text added: "1"

Commit message: Routing Work
Parts:
- moved SW45 1.52 mm to (83.0, 102.5), turned to 90 degrees
- moved R6 1.13 mm to (95.5, 98.6), turned to -90 degrees
- moved R7 1.13 mm to (201.7, 98.1), turned to -90 degrees
- moved C9 0.07 mm to (195.0, 102.5)
Connections:
- U1 pad 10: unconnected-(U1-PA0-Pad10) -> /SwitchClusterLeft/Column7
- U1 pad 11: unconnected-(U1-PA1-Pad11) -> /SwitchClusterLeft/Column6
- U1 pad 12: unconnected-(U1-PA2-Pad12) -> /SwitchClusterLeft/Column5
- U1 pad 13: unconnected-(U1-PA3-Pad13) -> /SwitchClusterLeft/Column4
- U1 pad 14: unconnected-(U1-PA4-Pad14) -> /SwitchClusterLeft/Column3
- U1 pad 15: unconnected-(U1-PA5-Pad15) -> /SwitchClusterLeft/Column2
- U1 pad 16: unconnected-(U1-PA6-Pad16) -> /SwitchClusterLeft/Column1
- U1 pad 34: unconnected-(U1-PA13-Pad34) -> /SwitchClusterLeft/Row3
- U1 pad 37: unconnected-(U1-PA14-Pad37) -> /SwitchClusterLeft/Row2
- U1 pad 38: unconnected-(U1-PA15-Pad38) -> /SwitchClusterLeft/Row1
- U3 pad 10: unconnected-(U3-PA0-Pad10) -> /SwitchClusterRight/Column7
- U3 pad 11: unconnected-(U3-PA1-Pad11) -> /SwitchClusterRight/Column6
- U3 pad 12: unconnected-(U3-PA2-Pad12) -> /SwitchClusterRight/Column5
- U3 pad 13: unconnected-(U3-PA3-Pad13) -> /SwitchClusterRight/Column4
- U3 pad 14: unconnected-(U3-PA4-Pad14) -> /SwitchClusterRight/Column3
- U3 pad 15: unconnected-(U3-PA5-Pad15) -> /SwitchClusterRight/Column2
- U3 pad 16: unconnected-(U3-PA6-Pad16) -> /SwitchClusterRight/Column1
- U3 pad 34: unconnected-(U3-PA13-Pad34) -> /SwitchClusterRight/Row3
- U3 pad 37: unconnected-(U3-PA14-Pad37) -> /SwitchClusterRight/Row2
- U3 pad 38: unconnected-(U3-PA15-Pad38) -> /SwitchClusterRight/Row1
Routing:
- net /SwitchClusterRight/Row1: track 0.00 -> 127.1 mm, vias 0 -> 10
- net /SwitchClusterLeft/Row3: track 0.00 -> 120.7 mm, vias 0 -> 8
- net /SwitchClusterLeft/Row2: track 0.00 -> 116.9 mm, vias 0 -> 10
- net /SwitchClusterRight/Row3: track 0.00 -> 113.2 mm, vias 0 -> 10
- net /SwitchClusterRight/Row2: track 0.00 -> 113.1 mm, vias 0 -> 10
- net /SwitchClusterLeft/Row1: track 0.00 -> 111.6 mm, vias 0 -> 4
- net /SwitchClusterRight/Column4: track 0.00 -> 44.5 mm
- net /SwitchClusterRight/Column3: track 0.00 -> 44.2 mm
- net /SwitchClusterRight/Column2: track 0.00 -> 44.2 mm
- net GND: track 0.00 -> 44.1 mm, vias 0 -> 10
- net /SwitchClusterRight/Column5: track 0.00 -> 44.1 mm
- net /SwitchClusterLeft/Column6: track 0.00 -> 44.0 mm
- net /SwitchClusterRight/Column6: track 0.00 -> 44.0 mm
- net /SwitchClusterRight/Column1: track 0.00 -> 44.0 mm
- net /SwitchClusterLeft/Column5: track 0.00 -> 44.0 mm
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- added copper zone on F.Cu, net GND

Commit message: more routing
Parts:
- added D44: LED, LED_SMD:LED_0805_2012Metric, B.Cu at (120.7, 113.5)
- added D45: LED, LED_SMD:LED_0805_2012Metric, F.Cu at (162.9, 47.8)
- added D46: LED, LED_SMD:LED_0805_2012Metric, B.Cu at (89.2, 110.9)
- added D47: LED, LED_SMD:LED_0805_2012Metric, B.Cu at (207.2, 99.2)
- added J8: Debug UART, Connector_PinHeader_2.54mm:PinHeader_1x04_P2.54mm_Vertical, F.Cu at (133.2, 46.0)
- added J9: Debug UART, Connector_PinHeader_2.54mm:PinHeader_1x04_P2.54mm_Vertical, F.Cu at (138.2, 45.5)
- added R10: 100R, Resistor_SMD:R_0402_1005Metric, B.Cu at (209.8, 100.0)
- added R3: 100R, Resistor_SMD:R_0402_1005Metric, B.Cu at (123.7, 113.5)
- added R4: 100R, Resistor_SMD:R_0402_1005Metric, F.Cu at (160.0, 48.0)
- added R9: 100R, Resistor_SMD:R_0402_1005Metric, B.Cu at (92.5, 112.5)
- moved R1 11.5 mm to (114.6, 86.5)
- moved R2 11.3 mm to (114.8, 88.8)
- moved C6 0.32 mm to (208.0, 102.2)
- moved C7 0.32 mm to (206.8, 102.2)
- moved C4 0.21 mm to (100.8, 108.2)
- moved C15 0.14 mm to (206.8, 106.2)
- moved C16 0.14 mm to (207.8, 106.2)
- moved C17 0.14 mm to (209.0, 106.2)
Connections:
- U1 pad 2: unconnected-(U1-PC13-Pad2) -> /PC13
- U1 pad 30: unconnected-(U1-PA9-Pad30) -> /TX
- U1 pad 31: unconnected-(U1-PA10-Pad31) -> /RX
- U1 pad 32: unconnected-(U1-PA11-Pad32) -> D-
- U1 pad 33: unconnected-(U1-PA12-Pad33) -> D+
- U3 pad 2: unconnected-(U3-PC13-Pad2) -> /PC13
- U3 pad 30: unconnected-(U3-PA9-Pad30) -> Net-(J9-Pin_2)
- U3 pad 31: unconnected-(U3-PA10-Pad31) -> Net-(J9-Pin_3)
Routing:
- net /SwitchClusterLeft/Row1: track 111.6 -> 214.7 mm, vias 4 -> 9
- net +3.3V: track 25.0 -> 127.2 mm, vias 0 -> 6
- net /SwitchClusterLeft/Column6: track 44.0 -> 107.5 mm, vias 0 -> 2
- net /BOOT1R: track 0.00 -> 52.6 mm, vias 0 -> 2
- net /SwitchClusterLeft/Row2: track 116.9 -> 169.3 mm, vias 10 -> 14
- net /BOOT0R: track 0.00 -> 48.6 mm, vias 0 -> 1
- net /SwitchClusterLeft/Row3: track 120.7 -> 166.8 mm
- net /SwitchClusterLeft/Column5: track 44.0 -> 87.3 mm, vias 0 -> 2
- net /SwitchClusterLeft/Column7: track 0.00 -> 42.6 mm
- net VBUS: track 7.59 -> 49.0 mm, vias 0 -> 2
- net /SwitchClusterLeft/Column1: track 44.0 -> 76.5 mm, vias 0 -> 2
- net /SwitchClusterLeft/Column4: track 44.0 -> 71.1 mm, vias 0 -> 2
- net GND: track 44.1 -> 63.3 mm, vias 10 -> 13
- net /SwitchClusterLeft/Column3: track 44.0 -> 60.6 mm, vias 0 -> 2
- net /SwitchClusterLeft/Column2: track 44.0 -> 57.3 mm, vias 0 -> 2
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- added copper zone on B.Cu, net +3.3V
- added copper zone on B.Cu, net VBUS

Commit message: routing done
Parts:
- removed J2, J7: AudioJack4, MyLibrary:Jack_3.5mm_CUI_SJ1-3524N_Horizontal
- D45, J8, J9, R4: moved to B.Cu
- moved J9 73.8 mm to (158.5, 116.5)
- moved J8 71.6 mm to (137.2, 117.5)
- moved D45 62.8 mm to (169.4, 110.2), turned to 180 degrees
- moved R4 59.8 mm to (169.7, 107.0)
- moved R2 20.3 mm to (134.9, 92.0), turned to 180 degrees
- moved R1 12.8 mm to (127.2, 85.0)
- moved R8 0.92 mm to (200.5, 111.7), turned to 90 degrees
- moved C9 0.34 mm to (195.2, 102.3)
- moved C4 0.25 mm to (100.8, 108.5)
Connections:
- net /RX renamed /RX_M
- net /TX renamed /TX_M
- C14 pad 1: /NRST -> /NRST_M
- C18 pad 1: /NRST -> /NRST_S
- D46 pad 2: /PC13 -> /PC13_M
- D47 pad 2: /PC13 -> /PC13_S
- J3 pad 2: /BOOT0R -> /BOOT0R_M
- J4 pad 2: /BOOT1R -> /BOOT1R_M
- J5 pad 2: /BOOT0R -> /BOOT0R_S
- J6 pad 2: /BOOT1R -> /BOOT1R_S
- J9 pad 2: Net-(J9-Pin_2) -> /RX_S
- J9 pad 3: Net-(J9-Pin_3) -> /TX_S
- R5 pad 1: /BOOT0R -> /BOOT0R_M
- R5 pad 2: /BOOT0 -> /BOOT0_M
- R6 pad 1: /BOOT1R -> /BOOT1R_M
- R6 pad 2: /BOOT1 -> /BOOT1_M
- R7 pad 1: /BOOT0R -> /BOOT0R_S
- R7 pad 2: /BOOT0 -> /BOOT0_S
- R8 pad 1: /BOOT1R -> /BOOT1R_S
- R8 pad 2: /BOOT1 -> /BOOT1_S
- SW43 pad 2: /NRST -> /NRST_S
- SW45 pad 2: /NRST -> /NRST_M
- U1 pad 2: /PC13 -> /PC13_M
- U1 pad 20: /BOOT1 -> /BOOT1_M
- U1 pad 44: /BOOT0 -> /BOOT0_M
- U1 pad 7: /NRST -> /NRST_M
- U3 pad 2: /PC13 -> /PC13_S
- U3 pad 20: /BOOT1 -> /BOOT1_S
- U3 pad 30: Net-(J9-Pin_2) -> /TX_S
- U3 pad 31: Net-(J9-Pin_3) -> /RX_S
- U3 pad 44: /BOOT0 -> /BOOT0_S
- U3 pad 7: /NRST -> /NRST_S
Routing:
- net /SwitchClusterRight/Row1: track 133.0 -> 241.7 mm, vias 10 -> 13
- net +3.3V: track 127.2 -> 200.8 mm, vias 6 -> 14
- net /SwitchClusterRight/Row2: track 114.1 -> 186.7 mm, vias 10 -> 13
- net /SwitchClusterRight/Column6: track 44.0 -> 113.2 mm, vias 0 -> 2
- net /SwitchClusterRight/Column7: track 0.00 -> 65.8 mm
- net /TX_M: track 0.00 -> 58.6 mm, vias 0 -> 1
- net /RX_M: track 0.00 -> 57.2 mm, vias 0 -> 1
- net /BOOT1R_S: track 0.00 -> 56.7 mm, vias 0 -> 2
- net /BOOT1R_M: track 0.00 -> 52.6 mm, vias 0 -> 2
- net /BOOT1R: track 52.6 -> 0.00 mm, vias 2 -> 0
- net /RX_S: track 0.00 -> 51.8 mm, vias 0 -> 1
- net /BOOT0R_S: track 0.00 -> 50.1 mm, vias 0 -> 1
- net /SwitchClusterRight/Column5: track 44.1 -> 93.1 mm, vias 0 -> 2
- net /BOOT0R_M: track 0.00 -> 48.7 mm, vias 0 -> 1
- net /BOOT0R: track 48.6 -> 0.00 mm, vias 1 -> 0
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
Commit message: fix rule checker errors and make BOM
Parts:
- moved R2 13.9 mm to (132.6, 78.2)
- moved R8 0.86 mm to (201.2, 111.2), turned to 180 degrees
- moved D47 0.25 mm to (207.2, 99.0)
Routing:
- net Net-(J1-CC2): track 6.47 -> 9.28 mm
- net /BOOT1R_S: track 56.7 -> 58.7 mm
Other:
- board size 260 x 100.9 mm -> 261 x 101.9 mm

Commit message: Add mount holes n stuff
Parts:
- removed the U1 at (95.0, 105.5)
- added H1: MountingHole, MountingHole:MountingHole_3mm, F.Cu at (220.2, 79.5)
- added H2: MountingHole, MountingHole:MountingHole_3mm, F.Cu at (74.8, 79.5)
- added H3: MountingHole, MountingHole:MountingHole_3mm, F.Cu at (112.8, 73.5)
- added H4: MountingHole, MountingHole:MountingHole_3mm, F.Cu at (182.2, 73.5)
- added H5: MountingHole, MountingHole:MountingHole_3mm, F.Cu at (36.8, 91.5)
- added H6: MountingHole, MountingHole:MountingHole_3mm, F.Cu at (259.8, 98.0)
- added H7: MountingHole, MountingHole:MountingHole_3mm, F.Cu at (124.8, 120.8)
- added H8: MountingHole, MountingHole:MountingHole_3mm, F.Cu at (167.8, 118.0)
- added U2: STM32F103C8Tx, Package_QFP:LQFP-48_7x7mm_P0.5mm, B.Cu at (95.0, 105.5)
- C13: renamed from C18; value 100n -> 100nF
- C14: value 100n -> 100nF
- U3: value STM32F103C6Tx -> STM32F103C8Tx
- renumbered C13 to C18, C6 to C2, C2 to C6, J3 to J2, J4 to J3, J5 to J4, J6 to J5, J8 to J6, J9 to J7, R6 to R10, R9 to R5, R10 to R6, R5 to R9, SW45 to SW44, U2 to U1
