File: PCB/Keyboard-PCB.kicad_pcb (KiCad board)
At the start: 2 copper layers, 261 x 101.9 mm, 141 parts, among them J1 USB_C_Receptacle_USB2.0_16P, J2 BOOT0, J3 BOOT1, J4 BOOT0, J5 BOOT1, J6 Debug UART, J7 Debug UART, SW1 SW_Push, SW10 SW_Push, SW11 SW_Push, SW12 SW_Push, SW13 SW_Push, SW14 SW_Push, SW15 SW_Push, SW16 SW_Push, SW17 SW_Push, SW18 SW_Push, SW19 SW_Push, SW2 SW_Push, SW20 SW_Push, SW21 SW_Push, SW22 SW_Push, SW23 SW_Push, SW24 SW_Push, SW25 SW_Push, SW26 SW_Push, SW27 SW_Push, SW28 SW_Push, SW29 SW_Push, SW3 SW_Push, SW30 SW_Push, SW31 SW_Push, SW32 SW_Push, SW33 SW_Push, SW34 SW_Push, SW35 SW_Push, SW36 SW_Push, SW37 SW_Push, SW38 SW_Push, SW39 SW_Push, SW4 SW_Push, SW40 SW_Push, SW41 SW_Push, SW42 SW_Push, SW43 SW_Push, SW44 SW_Push, SW5 SW_Push, SW6 SW_Push, SW7 SW_Push, SW8 SW_Push, SW9 SW_Push, U1 AMS1117-3.3, U2 STM32F103C8Tx, U3 STM32F103C8Tx

Commit message: Add more mounting holes and do some cad work
Parts:
- added H10: MountingHole, MountingHole:MountingHole_3mm, F.Cu at (239.2, 66.5)
- added H11: MountingHole, MountingHole:MountingHole_3mm, F.Cu at (74.8, 60.5)
- added H12: MountingHole, MountingHole:MountingHole_3mm, F.Cu at (192.2, 121.0)
- added H13: MountingHole, MountingHole:MountingHole_3mm, F.Cu at (102.8, 122.0)
- added H14: MountingHole, MountingHole:MountingHole_3mm, F.Cu at (202.8, 60.5)
- added H9: MountingHole, MountingHole:MountingHole_3mm, F.Cu at (55.8, 85.5)
- moved H1 20.8 mm to (93.8, 88.0)
- moved H2 19.0 mm to (112.8, 54.5)
- moved H3 19.0 mm to (36.8, 72.5)
- moved H5 6.18 mm to (221.8, 85.5)
- renumbered H2 to H1, H3 to H2, H5 to H3, H7 to H4, H1 to H5, H4 to H6, H6 to H7
Routing:
- net /SwitchClusterLeft/Row1: track 215.7 -> 214.0 mm
- net /SwitchClusterRight/Row1: track 241.7 -> 241.1 mm
